Commit message: restructured .urdf; added model.launch

File: main/urdf/wheatley_model.urdf (robot description, URDF)
Before this commit: robot Wheatley, 5 links, 4 joints
Links:
- removed link front
- removed link lWheel
- removed link rWheel
- removed link top
- added link front_marker; visual box size=0.01 0.01 0.01
- added link wheel_left; visual cylinder length=0.025 radius=0.05
- added link wheel_right; visual cylinder length=0.025 radius=0.05
- link base_link: geometry visual box size=0.165 0.075 0.175; visual cylinder length=0.08 radius=0.1125
Joints:
- removed joint base_to_right_leg
- removed joint show_front
- added joint base_to_front_marker: type fixed, parent base_link, child front_marker, origin xyz=0 0.111 0.105
- joint base_to_left_wheel: child lWheel -> wheel_left
- joint base_to_right_wheel: child rWheel -> wheel_right

Commit message: base.launch now starts arduino and motorcontroller aswell

File: main/urdf/wheatley_model.urdf (robot description, URDF)
Before this commit: robot Wheatley, 4 links, 3 joints
Links:
- removed link base_link
- added link robot; visual box size=0.165 0.075 0.175; visual cylinder length=0.08 radius=0.1125
Joints:
- removed joint base_to_front_marker
- removed joint base_to_left_wheel
- removed joint base_to_right_wheel
- added joint robot_to_front_marker: type fixed, parent robot, child front_marker, origin xyz=0 0.111 0.105
- added joint robot_to_left_wheel: type fixed, parent robot, child wheel_left, origin xyz=-0.112 0 0.05
- added joint robot_to_right_wheel: type fixed, parent robot, child wheel_right, origin xyz=0.112 0 0.05

Commit message: now publishing /sensors/ir/points
forward is now positive on the x-axis, and left is positive on the y-axis
added Header to Distance.msg
distances in Distance.msg are now in m instead of cm
moved /sensors/distance to /sensors/ir/distances
added camera_link in .urdf and removed tf_robot_to_camera.launch
added joint types to .urdf

File: main/urdf/wheatley_model.urdf (robot description, URDF)
Before this commit: robot Wheatley, 4 links, 3 joints
Links:
- removed link front_marker
- added link camera_link; visual box size=0.0465 0.18 0.0245
- added link ir_front
- added link ir_left_front
- added link ir_left_rear
- added link ir_rear
- added link ir_right_front
- added link ir_right_rear
- link robot: geometry visual box size=0.075 0.165 0.175; visual cylinder length=0.08 radius=0.1125
- link wheel_left: geometry visual cylinder length=0.026 radius=0.05
- link wheel_right: geometry visual cylinder length=0.026 radius=0.05
Joints:
- removed joint robot_to_front_marker
- added joint robot_to_camera_link: type revolute, parent robot, child camera_link, origin xyz=0.02 0 0.295 rpy=0 0.6 0, axis 0 1 0, limit lower=-0.785 upper=0.785 effort=0 velocity=0
- added joint robot_to_ir_front: type fixed, parent robot, child ir_front, origin xyz=0.112 0 0.0825 rpy=0 0 0
- added joint robot_to_ir_left_front: type fixed, parent robot, child ir_left_front, origin xyz=0.082 0.119 0.0825 rpy=0 0 1.57075
- added joint robot_to_ir_left_rear: type fixed, parent robot, child ir_left_rear, origin xyz=-0.082 0.119 0.0825 rpy=0 0 1.57075
- added joint robot_to_ir_rear: type fixed, parent robot, child ir_rear, origin xyz=-0.112 0 0.0825 rpy=0 0 3.14159
- added joint robot_to_ir_right_front: type fixed, parent robot, child ir_right_front, origin xyz=0.082 -0.119 0.0825 rpy=0 0 -1.57075
- added joint robot_to_ir_right_rear: type fixed, parent robot, child ir_right_rear, origin xyz=-0.082 -0.119 0.0825 rpy=0 0 -1.57075
- joint robot_to_left_wheel: axis (none) -> 1 0 0; origin xyz=-0.112 0 0.05 -> xyz=0 0.0925 0.05 rpy=0 0 1.57075; type fixed -> continuous
- joint robot_to_right_wheel: axis (none) -> 1 0 0; origin xyz=0.112 0 0.05 -> xyz=0 -0.0925 0.05 rpy=0 0 -1.57075; type fixed -> continuous

Commit message: Fixed executor_node.cpp

File: main/urdf/wheatley_model.urdf (robot description, URDF)
Before this commit: robot Wheatley, 10 links, 9 joints
Joints:
- joint robot_to_camera_link: origin xyz=0.02 0 0.295 rpy=0 0.6 0 -> xyz=0.03 0 0.26 rpy=0.02 0.52 0

Commit message: moved camera_link in .urdf

File: main/urdf/wheatley_model.urdf (robot description, URDF)
Before this commit: robot Wheatley, 10 links, 9 joints
Links:
- link robot: geometry visual box size=0.075 0.165 0.155; visual cylinder length=0.08 radius=0.1125
Joints:
- joint robot_to_camera_link: origin xyz=0.03 0 0.26 rpy=0.02 0.52 0 -> xyz=0.00 0.05 0.26 rpy=0.02 0.52 0

Commit message: STAGING PULL (johntu)

File: main/urdf/wheatley_model.urdf (robot description, URDF)
Before this commit: robot Wheatley, 10 links, 9 joints
Joints:
- joint robot_to_camera_link: origin xyz=0.00 0.05 0.26 rpy=0.02 0.52 0 -> xyz=0.00 0.05 0.25 rpy=0.02 0.52 0

Commit message: Moved camera to the front, because of wrong distance measurements

File: main/urdf/wheatley_model.urdf (robot description, URDF)
Before this commit: robot Wheatley, 10 links, 9 joints
Joints:
- joint robot_to_camera_link: origin xyz=0.00 0.05 0.25 rpy=0.02 0.52 0 -> xyz=0.05 0.065 0.26 rpy=0 0.52 0

Commit message: Adjusted the camera rotation

File: main/urdf/wheatley_model.urdf (robot description, URDF)
Before this commit: robot Wheatley, 10 links, 9 joints
Joints:
- joint robot_to_camera_link: origin xyz=0.05 0.065 0.26 rpy=0 0.52 0 -> xyz=0.05 0.065 0.26 rpy=0 0.52 -0.034
